File: Hardware/Hardware.kicad_pcb (KiCad board)
At the start: 2 copper layers, 29 parts, among them J1 USB_C_Receptacle_USB2.0_16P, J2 Conn_01x06, J3 Conn_01x04, Q1 BSS138, Q2 BSS138, U2 CH340C, U4 ESP32-WROOM-32, U5 AMS1117-3.3

Commit message: move usb C
Parts:
- moved C15 70.8 mm to (91.3, 50.6), turned to -90 degrees
- moved D4 49.7 mm to (149.8, 53.4)
- moved J2 27.6 mm to (117.3, 50.3)
- moved U5 21.7 mm to (82.8, 52.6), turned to 90 degrees
- moved Q1 13.3 mm to (88.4, 62.9), turned to 180 degrees
- moved Q2 13.2 mm to (88.3, 67.7), turned to 180 degrees
- moved J1 10.3 mm to (70.4, 65.4)
- moved U2 9.94 mm to (81.8, 64.2)
- moved C33 6.70 mm to (87.8, 54.3), turned to -90 degrees
Connections:
- C15 pad 2: +BATT -> +3V3
- C32 pad 2: +BATT -> +5V
- C33 pad 2: +BATT -> +5V

Commit message: end position pcb
Parts:
- removed D2: D_Schottky, Diode_SMD:D_0805_2012Metric
- added R8: R_Small, Resistor_SMD:R_0603_1608Metric, F.Cu at (127.5, 51.7)
- added R9: R_Small, Resistor_SMD:R_0603_1608Metric, F.Cu at (127.5, 70.0)
- moved C32 86.9 mm to (74.7, 54.7)
- moved R3 83.5 mm to (73.8, 58.8)
- moved R2 83.3 mm to (73.8, 57.0), turned to 180 degrees
- moved C7 61.3 mm to (81.6, 70.4)
- moved C8 53.2 mm to (81.8, 58.1), turned to 180 degrees
- moved D4 51.7 mm to (100.6, 69.2)
- moved C6 50.7 mm to (87.8, 58.4), turned to -90 degrees
- moved C5 47.1 mm to (91.3, 54.7), turned to -90 degrees
- moved C9 46.0 mm to (91.4, 62.8), turned to -90 degrees
- moved J3 43.3 mm to (134.8, 56.3)
- moved R6 35.5 mm to (103.8, 69.2), turned to 180 degrees
- moved D3 29.4 mm to (131.6, 60.0), turned to -90 degrees
- moved R5 26.8 mm to (117.2, 66.0), turned to 180 degrees
- moved R4 17.2 mm to (122.6, 55.4)
- moved R7 16.1 mm to (131.6, 63.2), turned to 90 degrees
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- renumbered BOTTOM1 to PROGRAM1
Connections:
- J1 pad A4: Net-(D2-K) -> +5V
- J1 pad A9: Net-(D2-K) -> +5V
- J1 pad B4: Net-(D2-K) -> +5V
- J1 pad B9: Net-(D2-K) -> +5V
- PROGRAM1 pad 1: unconnected-(BOTTOM1-Pad1) -> BTN2
- PROGRAM1 pad 2: unconnected-(BOTTOM1-Pad2) -> GND
- TOP1 pad 1: unconnected-(TOP1-Pad1) -> BTN1
- TOP1 pad 2: unconnected-(TOP1-Pad2) -> GND
- U4 pad 23: unconnected-(U4-IO15-Pad23) -> BTN1
- U4 pad 27: unconnected-(U4-IO16-Pad27) -> BTN2

Commit message: finish pcb wiring
Parts:
- moved D3 8.98 mm to (137.7, 66.6), turned to 180 degrees
- moved R7 4.47 mm to (134.5, 66.6), turned to 0 degrees
- moved R2 2.01 mm to (74.0, 59.0)
- moved R3 1.81 mm to (74.0, 57.0)
Connections:
- U4 pad 36: SWCLK -> SWDIO
- U4 pad 37: SWDIO -> SWCLK
Routing:
- net +3V3: track 0.00 -> 146.8 mm, vias 0 -> 4
- net +5V: track 0.00 -> 78.1 mm, vias 0 -> 3
- net ESP32_IO0: track 0.00 -> 50.4 mm
- net ESP32_EN: track 0.00 -> 49.8 mm, vias 0 -> 3
- net RX-PROG: track 0.00 -> 46.1 mm, vias 0 -> 2
- net TX-PROG: track 0.00 -> 45.2 mm, vias 0 -> 2
- net Net-(U4-IO13): track 0.00 -> 39.4 mm
- net BTN2: track 0.00 -> 31.0 mm
- net SWDIO: track 0.00 -> 27.1 mm, vias 0 -> 1
- net SWCLK: track 0.00 -> 26.6 mm, vias 0 -> 1
- net BTN1: track 0.00 -> 24.9 mm, vias 0 -> 2
- net Net-(Q1-S): track 0.00 -> 19.0 mm
- net Net-(U4-IO12): track 0.00 -> 15.5 mm, vias 0 -> 2
- net Net-(J1-CC2): track 0.00 -> 14.3 mm
- net Net-(J1-CC1): track 0.00 -> 8.24 mm
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- added copper zone on B.Cu, net GND
- added copper zone on F.Cu, net GND
Other:
- board outline added: 72 x 25 mm
- board text added: "3.3 SWCLK SWDIO GND"
