File: Hardware/Hardware.kicad_sch (KiCad schematic)
At the start: 29 parts, among them J1 USB_C_Receptacle_USB2.0_16P, J2 Conn_01x06, J3 Conn_01x04, Q1 BSS138, Q2 BSS138, U2 CH340C, U4 ESP32-WROOM-32, U5 AMS1117-3.3

Commit message: end position pcb
Parts:
- removed D2: D_Schottky, Diode_SMD:D_0805_2012Metric, symbol Device:D_Schottky
- added R8, R9: R_Small, Resistor_SMD:R_0603_1608Metric, symbol Device:R_Small
- renumbered BOTTOM1 to PROGRAM1
Connections:
- net +3V3: now also R8.1, R9.1
- net +5V: now also J1.A4 (VBUS), J1.A9 (VBUS), J1.B4 (VBUS), J1.B9 (VBUS)
- net GND: now also PROGRAM1.2, TOP1.2
- net BTN1: now reaches TOP1.1
- net BTN1: now also U4.23 (IO15), R9.2
- net BTN2: now reaches U4.27 (IO16)
- net BTN2: now also PROGRAM1.1, R8.2
Other:
- moved on the sheet: PROGRAM1, TOP1

Commit message: finish pcb wiring
Connections:
- net SWCLK: now also U4.37 (IO23); no longer U4.36 (IO22)
- net SWDIO: now also U4.36 (IO22); no longer U4.37 (IO23)
Changed lines of the file:
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@@
+		)
+	)
+	(global_label "SWCLK"
+		(shape input)
+		(at 110.49 111.76 0)
+		(fields_autoplaced yes)
+		(effects
+			(font
+				(size 1.27 1.27)
+			)
+			(justify left)
+		)
+		(property "Intersheetrefs" "${INTERSHEET_REFS}"
+			(at 119.7042 111.76 0)
+			(hide yes)
+			(show_name no)
+			(do_not_autoplace no)
+			(effects
+				(font
+					(size 1.27 1.27)
+				)
+				(justify left)
+			)
 		)
 	)
@@
 		(property "Intersheetrefs" "${INTERSHEET_REFS}"
 			(at 122.4861 104.14 0)
-			(hide yes)
-			(show_name no)
-			(do_not_autoplace no)
-			(effects
-				(font
-					(size 1.27 1.27)
-				)
-				(justify left)
-			)
-		)
-	)
-	(global_label "SWDIO"
-		(shape input)
-		(at 110.49 111.76 0)
-		(fields_autoplaced yes)
-		(effects
-			(font
-				(size 1.27 1.27)
-			)
-			(justify left)
-		)
-		(property "Intersheetrefs" "${INTERSHEET_REFS}"
-			(at 119.3414 111.76 0)
 			(hide yes)
 			(show_name no)
@@
 		)
 	)
+	(global_label "SWDIO"
+		(shape input)
+		(at 110.49 109.22 0)
+		(fields_autoplaced yes)
+		(effects
+			(font
+				(size 1.27 1.27)
+			)
+			(justify left)
+		)
+		(property "Intersheetrefs" "${INTERSHEET_REFS}"
+			(at 119.3414 109.22 0)
+			(hide yes)
+			(show_name no)
+			(do_not_autoplace no)
+			(effects
+				(font
+					(size 1.27 1.27)
+				)
+				(justify left)
+			)
+		)
+	)
 	(global_label "TX-PROG"
 		(shape input)
@@
 			(hide yes)
 			(show_name no)
-			(do_not_autoplace no)
-			(effects
-				(font
-					(size 1.27 1.27)
-				)
-				(justify left)
-			)
-		)
-	)
-	(global_label "SWCLK"
-		(shape input)
-		(at 110.49 109.22 0)
-		(fields_autoplaced yes)
-		(effects
-			(font
-				(size 1.27 1.27)
-			)
-			(justify left)
-		)
-		(property "Intersheetrefs" "${INTERSHEET_REFS}"
-			(at 119.7042 109.22 0)
-			(hide yes)
-			(show_name no)
